Commit message: Resolved what seemed to be friection inconsistency
It was an issue with the acceleration limits, removing the limits resolved the issue

File: description/gazebo_control.xacro (robot description, xacro)
@@ -1,4 +1,5 @@
 <?xml version="1.0"?>
 <robot xmlns:xacro="http://www.ros.org/wiki/xacro">
+    <xacro:include filename="measurements.xacro" />
     <gazebo>
         <plugin name="gz::sim::systems::DiffDrive" filename="gz-sim-diff-drive-system">
@@ -6,9 +7,9 @@
             <left_joint>left_wheel_joint</left_joint>
             <right_joint>right_wheel_joint</right_joint>
-            <wheel_separation>0.297</wheel_separation>
-            <wheel_radius>0.033</wheel_radius>
+            <wheel_separation>${chassis_width}</wheel_separation>
+            <wheel_radius>${wheel_radius}</wheel_radius>
             <!-- Limits -->
-            <!-- <max_wheel_torque>200</max_wheel_torque> -->
-            <max_linear_acceleration>0.33</max_linear_acceleration>
+            <max_wheel_torque>200</max_wheel_torque>
+            <!-- <max_linear_acceleration>0.2</max_linear_acceleration> -->
             <!-- Input -->
             <topic>cmd_vel</topic>

File: description/robot.urdf.xacro (robot description, xacro)
@@ -3,3 +3,4 @@
 <xacro:include filename="robot_core.xacro" />
 <xacro:include filename="gazebo_control.xacro" />
+<!-- <xacro:include filename="ros2_control.xacro" /> -->
 </robot>

File: description/robot_core.xacro (robot description, xacro)
@@ -1,114 +1,204 @@
 <?xml version="1.0"?>
 <robot xmlns:xacro="http://www.ros.org/wiki/xacro">
-<xacro:include filename="inertial_macros.xacro" />
-<material name="white">
-    <color rgba="1 1 1 1" />
-</material>
-<material name="black">
-    <color rgba="0 0 0 1" />
-</material>
-<material name="orange">
-    <color rgba="1 0.3 0.1 1" />
-</material>
-<material name="blue">
-    <color rgba="0.2 0.2 1 1" />
-</material>
-<!-- BASE LINK-->
-<link name="base_link">
-</link>
-<!-- CHASSIS LINK-->
-<joint name="chassis_joint" type="fixed">
-    <parent link="base_link" />
-    <child link="chassis" />
-    <origin xyz="-0.1 0 0" />
-</joint>
-<link name="chassis">
-    <visual>
-        <origin xyz="0.15 0 0.075" />
-        <geometry>
-            <box size="0.3 0.3 0.15" />
-        </geometry>
-        <material name="white" />
-    </visual>
-    <collision>
-        <origin xyz="0.15 0 0.075" />
-        <geometry>
-            <box size="0.3 0.3 0.15" />
-        </geometry>
-    </collision>
-    <xacro:inertial_box mass="0.5" x="0.3" y="0.3" z="0.15">
-        <origin xyz="0.15 0 0.075" rpy="0 0 0" />
-    </xacro:inertial_box>
-</link>
-<gazebo reference="chassis">
-    <material>Gazebo/White</material>
-</gazebo>
-<!-- LEFT WHEEL LINK-->
-<joint name="left_wheel_joint" type="continuous">
-    <parent link="base_link" />
-    <child link="left_wheel" />
-    <origin xyz="0 0.175 0" rpy="-${pi/2} 0 0" />
-    <axis xyz="0 0 1" />
-</joint>
-<link name="left_wheel">
-    <visual>
-        <geometry>
-            <cylinder radius="0.05" length="0.04" />
-        </geometry>
-        <material name="blue" />
-    </visual>
-    <collision>
-        <geometry>
-            <cylinder radius="0.05" length="0.04" />
-        </geometry>
-    </collision>
-    <xacro:inertial_cylinder mass="0.1" length="0.04" radius="0.05">
-        <origin xyz="0 0 0" rpy="0 0 0" />
-    </xacro:inertial_cylinder>
-</link>
-<!-- RIGHT WHEEL LINK-->
-<joint name="right_wheel_joint" type="continuous">
-    <parent link="base_link" />
-    <child link="right_wheel" />
-    <origin xyz="0 -0.175 0" rpy="${pi/2} 0 0" />
-    <axis xyz="0 0 -1" />
-</joint>
-<link name="right_wheel">
-    <visual>
-        <geometry>
-            <cylinder radius="0.05" length="0.04" />
-        </geometry>
-        <material name="blue" />
-    </visual>
-    <collision>
-        <geometry>
-            <cylinder radius="0.05" length="0.04" />
-        </geometry>
-    </collision>
-    <xacro:inertial_cylinder mass="0.1" length="0.04" radius="0.05">
-        <origin xyz="0 0 0" rpy="0 0 0" />
-    </xacro:inertial_cylinder>
-</link>
-<!-- CASTER WHEEL LINK-->
-<joint name="caster_wheel_link" type="fixed">
-    <parent link="chassis" />
-    <child link="caster_wheel" />
-    <origin xyz="0.25 0 0" />
-</joint>
-<link name="caster_wheel">
-    <visual>
-        <geometry>
-            <sphere radius="0.05" />
-        </geometry>
-        <material name="black" />
-    </visual>
-    <collision>
-        <geometry>
-            <sphere radius="0.05" />
-        </geometry>
-    </collision>
-    <xacro:inertial_sphere mass="0.1" radius="0.05">
-        <origin xyz="0 0 0" rpy="0 0 0" />
-    </xacro:inertial_sphere>
-</link>
+    <xacro:include filename="inertial_macros.xacro" />
+    <xacro:include filename="measurements.xacro" />
+    <material name="white">
+        <color rgba="1 1 1 1" />
+    </material>
+    <material name="black">
+        <color rgba="0 0 0 1" />
+    </material>
+    <material name="orange">
+        <color rgba="1 0.3 0.1 1" />
+    </material>
+    <material name="blue">
+        <color rgba="0.2 0.2 1 1" />
+    </material>
+    <!-- BASE LINK-->
+    <link name="base_link">
+    </link>
+    <!-- CHASSIS LINK-->
+    <joint name="chassis_joint" type="fixed">
+        <parent link="base_link" />
+        <child link="chassis" />
+        <!-- <origin xyz="${-wheel_offset_x} 0 0" /> -->
+        <origin xyz="0 0 ${chassis_height/2}" />
+    </joint>
+    <link name="chassis">
+        <visual>
+            <!-- <origin xyz="${chassis_length/2} 0 ${chassis_height/2}" /> -->
+            <geometry>
+                <box size="${chassis_length} ${chassis_width} ${chassis_height}" />
+            </geometry>
+            <material name="white" />
+        </visual>
+        <collision>
+            <!-- <origin xyz="${chassis_length/2} 0 ${chassis_height/2}" /> -->
+            <geometry>
+                <box size="${chassis_length} ${chassis_width} ${chassis_height}" />
+            </geometry>
+        </collision>
+        <xacro:inertial_box mass="${chassis_mass}" x="${chassis_length}" y="${chassis_width}" z="${chassis_height}">
+            <!-- <origin xyz="${chassis_length/2} 0 ${chassis_height/2}" rpy="0 0 0" /> -->
+            <origin xyz="0 0 0" rpy="0 0 0" />
+        </xacro:inertial_box>
+    </link>
+    <!-- LEFT WHEEL LINK-->
+    <joint name="left_wheel_joint" type="continuous">
+        <parent link="base_link" />
+        <child link="left_wheel" />
+        <origin xyz="0 ${wheel_offset_y} 0" rpy="-${pi/2} 0 0" />
+        <axis xyz="0 0 1" />
+    </joint>
+    <link name="left_wheel">
+        <visual>
+            <geometry>
+                <cylinder radius="${wheel_radius}" length="${wheel_thickness}" />
+            </geometry>
+            <material name="orange" />
+        </visual>
+        <collision>
+            <geometry>
+                <cylinder radius="${wheel_radius}" length="${wheel_thickness}" />
+            </geometry>
+        </collision>
+        <xacro:inertial_cylinder mass="${wheel_mass}" length="${wheel_thickness}" radius="${wheel_radius}">
+            <origin xyz="0 0 0" rpy="0 0 0" />
+        </xacro:inertial_cylinder>
+    </link>
+    <!-- <joint name="left_wheel_joint" type="continuous">
+        <parent link="base_link" />
+        <child link="left_wheel" />
+        <origin xyz="0 ${wheel_offset_y} 0" rpy="-${pi/2} 0 0" />
+        <axis xyz="0 0 1" />
+    </joint>
+    <link name="left_wheel">
+        <visual>
+            <geometry>
+                <sphere radius="${wheel_radius}" />
+            </geometry>
+            <material name="orange" />
+        </visual>
+        <collision>
+            <geometry>
+                <cylinder radius="${wheel_radius}" />
+            </geometry>
+        </collision>
+        <xacro:inertial_sphere mass="${wheel_mass}" radius="${wheel_radius}">
+            <origin xyz="0 0 0" rpy="0 0 0" />
+        </xacro:inertial_sphere>
+    </link> -->
+    <!-- RIGHT WHEEL LINK-->
+    <joint name="right_wheel_joint" type="continuous">
+        <parent link="base_link" />
+        <child link="right_wheel" />
+        <origin xyz="0 ${-wheel_offset_y} 0" rpy="${pi/2} 0 0" />
+        <axis xyz="0 0 -1" />
+    </joint>
+    <link name="right_wheel">
+        <visual>
+            <geometry>
+                <cylinder radius="${wheel_radius}" length="${wheel_thickness}" />
+            </geometry>
+            <material name="blue" />
+        </visual>
+        <collision>
+            <geometry>
+                <cylinder radius="${wheel_radius}" length="${wheel_thickness}" />
+            </geometry>
+        </collision>
+        <xacro:inertial_cylinder mass="${wheel_mass}" length="${wheel_thickness}" radius="${wheel_radius}">
+            <origin xyz="0 0 0" rpy="0 0 0" />
+        </xacro:inertial_cylinder>
+    </link>
+    <!-- <joint name="right_wheel_joint" type="continuous">
+        <parent link="base_link" />
+        <child link="right_wheel" />
+        <origin xyz="0 ${-wheel_offset_y} 0" rpy="${pi/2} 0 0" />
+        <axis xyz="0 0 -1" />
+    </joint>
+    <link name="right_wheel">
+        <visual>
+            <geometry>
+                <sphere radius="${wheel_radius}" />
+            </geometry>
+            <material name="blue" />
+        </visual>
+        <collision>
+            <geometry>
+                <cylinder radius="${wheel_radius}" />
+            </geometry>
+        </collision>
+        <xacro:inertial_sphere mass="${wheel_mass}" radius="${wheel_radius}">
+            <origin xyz="0 0 0" rpy="0 0 0" />
+        </xacro:inertial_sphere>
+    </link> -->
+    <!-- FRONT CASTER WHEEL LINK-->
+    <joint name="front_caster_wheel_joint" type="fixed">
+        <parent link="base_link" />
+        <child link="front_caster_wheel" />
+        <origin xyz="${caster_wheel_offset_x} 0 0" />
+    </joint>
+    <link name="front_caster_wheel">
+        <visual>
+            <geometry>
+                <sphere radius="${caster_wheel_radius}" />
+            </geometry>
+            <material name="black" />
+        </visual>
+        <collision>
+            <geometry>
+                <sphere radius="${caster_wheel_radius}" />
+            </geometry>
+        </collision>
+        <xacro:inertial_sphere mass="${caster_wheel_mass}" radius="${caster_wheel_radius}">
+            <origin xyz="0 0 0" rpy="0 0 0" />
+        </xacro:inertial_sphere>
+    </link>
+    <gazebo reference="front_caster_wheel">
+        <collision>
+            <surface>
+                <friction>
+                    <ode>
+                        <mu>1.0</mu> <!-- value range 0.0 to 1.0 -->
+                        <mu2>0.5</mu2> <!-- value range 0.0 to 1.0 -->
+                    </ode>
+                </friction>
+            </surface>
+        </collision>
+    </gazebo>
+    <!-- REAR CASTER WHEEL LINK-->
+    <joint name="rear_caster_wheel_joint" type="fixed">
+        <parent link="base_link" />
+        <child link="rear_caster_wheel" />
+        <origin xyz="${-caster_wheel_offset_x} 0 0" />
+    </joint>
+    <link name="rear_caster_wheel">
+        <visual>
+            <geometry>
+                <sphere radius="${caster_wheel_radius}" />
+            </geometry>
+            <material name="black" />
+        </visual>
+        <collision>
+            <geometry>
+                <sphere radius="${caster_wheel_radius}" />
+            </geometry>
+        </collision>
+        <xacro:inertial_sphere mass="${caster_wheel_mass}" radius="${caster_wheel_radius}">
+            <origin xyz="0 0 0" rpy="0 0 0" />
+        </xacro:inertial_sphere>
+    </link>
+    <gazebo reference="rear_caster_wheel">
+        <collision>
+            <surface>
+                <friction>
+                    <ode>
+                        <mu>0.01</mu> <!-- value range 0.0 to 1.0 -->
+                        <mu2>0.01</mu2> <!-- value range 0.0 to 1.0 -->
+                    </ode>
+                </friction>
+            </surface>
+        </collision>
+    </gazebo>
 </robot>

File: description/ros2_control.xacro (robot description, xacro)
@@ -1,3 +1,3 @@
-<!-- <?xml version="1.0"?>
+<?xml version="1.0"?>
 <robot xmlns:xacro="http://www.ros.org/wiki/xacro">
     <xacro:unless value="$(arg sim_mode)">
@@ -56,7 +56,7 @@
     <gazebo>
         <plugin name="gz_ros2_control::GazeboSimROS2ControlPlugin" filename="libgz_ros2_control-system.so">
-            <parameters>$(find articubot_one)/config/my_controllers.yaml</parameters>
-            <parameters>$(find articubot_one)/config/gaz_ros2_ctl_use_sim.yaml</parameters>
+            <parameters>$(find my_bot)/config/my_controllers.yaml</parameters>
+            <parameters>$(find my_bot)/config/gaz_ros2_ctl_use_sim.yaml</parameters>
         </plugin>
     </gazebo>
-</robot> -->
+</robot>

Commit message: the failed attempt at implementing ros2control

File: description/gazebo_control.xacro (robot description, xacro)
@@ -3,5 +3,5 @@
     <xacro:include filename="measurements.xacro" />
     <gazebo>
-        <plugin name="gz::sim::systems::DiffDrive" filename="gz-sim-diff-drive-system">
+        <plugin name="diff_drive" filename="libgazebo_ros_diff_drive.so">
             <!-- Wheel Information -->
             <left_joint>left_wheel_joint</left_joint>
@@ -12,18 +12,10 @@
             <max_wheel_torque>200</max_wheel_torque>
             <!-- <max_linear_acceleration>0.2</max_linear_acceleration> -->
-            <!-- Input -->
-            <topic>cmd_vel</topic>
             <!-- Output -->
-            <frame_id>odom</frame_id>
-            <child_frame_id>base_link</child_frame_id>
-            <odom_topic>odom</odom_topic>
-            <odom_publisher_frequency>30</odom_publisher_frequency>
-            <tf_topic>/tf</tf_topic>
-        </plugin>
-        <plugin filename="gz-sim-joint-state-publisher-system"
-            name="gz::sim::systems::JointStatePublisher">
-            <topic>joint_states</topic>
-            <joint_name>left_wheel_joint</joint_name>
-            <joint_name>right_wheel_joint</joint_name>
+            <odometry_frame>odom</odometry_frame>
+            <robot_base_frame>base_link</robot_base_frame>
+            <publish_odom>true</publish_odom>
+            <publish_odom_tf>true</publish_odom_tf>
+            <publish_wheel_tf>true</publish_wheel_tf>
         </plugin>
     </gazebo>

File: description/robot.urdf.xacro (robot description, xacro)
@@ -2,5 +2,5 @@
 <robot xmlns:xacro="http://www.ros.org/wiki/xacro"  name="robot">
 <xacro:include filename="robot_core.xacro" />
-<xacro:include filename="gazebo_control.xacro" />
-<!-- <xacro:include filename="ros2_control.xacro" /> -->
+<!-- <xacro:include filename="gazebo_control.xacro" /> -->
+<xacro:include filename="ros2_control.xacro" />
 </robot>

File: description/ros2_control.xacro (robot description, xacro)
@@ -1,61 +1,38 @@
 <?xml version="1.0"?>
 <robot xmlns:xacro="http://www.ros.org/wiki/xacro">
-    <xacro:unless value="$(arg sim_mode)">
-        <ros2_control name="RealRobot" type="system">
-            <hardware>
-                <plugin>diffdrive_arduino/DiffDriveArduino</plugin>
-                <param name="left_wheel_name">left_wheel_joint</param>
-                <param name="right_wheel_name">right_wheel_joint</param>
-                <param name="loop_rate">30</param>
-                <param name="device">/dev/ttyUSB0</param>
-                <param name="baud_rate">57600</param>
-                <param name="timeout">1000</param>
-                <param name="enc_counts_per_rev">3436</param>
-            </hardware>
-            <joint name="left_wheel_joint">
-                <command_interface name="velocity">
-                    <param name="min">-10</param>
-                    <param name="max">10</param>
-                </command_interface>
-                <state_interface name="velocity"/>
-                <state_interface name="position"/>
-            </joint>
-            <joint name="right_wheel_joint">
-                <command_interface name="velocity">
-                    <param name="min">-10</param>
-                    <param name="max">10</param>
-                </command_interface>
-                <state_interface name="velocity"/>
-                <state_interface name="position"/>
-            </joint>
-        </ros2_control>
-    </xacro:unless>
-    <xacro:if value="$(arg sim_mode)">
-        <ros2_control name="GazeboSystem" type="system">
-            <hardware>
-                <plugin>gz_ros2_control/GazeboSystem</plugin>
-            </hardware>
-            <joint name="left_wheel_joint">
-                <command_interface name="velocity">
-                    <param name="min">-10</param>
-                    <param name="max">10</param>
-                </command_interface>
-                <state_interface name="velocity"/>
-                <state_interface name="position"/>
-            </joint>
-            <joint name="right_wheel_joint">
-                <command_interface name="velocity">
-                    <param name="min">-10</param>
-                    <param name="max">10</param>
-                </command_interface>
-                <state_interface name="velocity"/>
-                <state_interface name="position"/>
-            </joint>
-        </ros2_control>
-    </xacro:if>
+    <ros2_control name="IgnitionSystem" type="system">
+        <hardware>
+            <!-- <plugin>gazebo_ros2_control/GazeboSystem</plugin>   -->
+            <plugin>ign_ros2_control/IgnitionSystem</plugin>
+        </hardware>
+        <joint name="left_wheel_joint">
+            <command_interface name="velocity">
+                <param name="min">-10</param>
+                <param name="max">10</param>
+            </command_interface>
+            <state_interface name="velocity"/>
+            <state_interface name="position"/>
+        </joint>
+        <joint name="right_wheel_joint">
+            <command_interface name="velocity">
+                <param name="min">-10</param>
+                <param name="max">10</param>
+            </command_interface>
+            <state_interface name="velocity"/>
+            <state_interface name="position"/>
+        </joint>
+    </ros2_control>
+    <!-- <gazebo>
+        <plugin filename="libignition_ros2_control.so" name="ign_ros2_control">
+        <robot_param>robot_description</robot_param>
+        <robot_param_node>robot_state_publisher</robot_param_node>
+        <parameters>$(find my_bot)/config/my_controllers.yaml</parameters>
+        </plugin>
+    </gazebo> -->
     <gazebo>
-        <plugin name="gz_ros2_control::GazeboSimROS2ControlPlugin" filename="libgz_ros2_control-system.so">
+        <plugin filename="ign_ros2_control-system" name="ign_ros2_control::IgnitionROS2ControlPlugin">
+            <robot_param>robot_description</robot_param>
+            <robot_param_node>robot_state_publisher</robot_param_node>
             <parameters>$(find my_bot)/config/my_controllers.yaml</parameters>
-            <parameters>$(find my_bot)/config/gaz_ros2_ctl_use_sim.yaml</parameters>
         </plugin>
     </gazebo>
